File: pcb/ledPower.brd (EAGLE design)
At the start: 160 x 100 mm, 15 parts, among them X1 DG3XX-04-0.5, X2 DG3XX-02-5.0

Commit message: change sizes
Parts:
- moved R1 1.80 mm to (16.5, 16.5)
- moved C5 1.80 mm to (22.9, 5.08)
- moved X1 1.80 mm to (6.35, 15.2)
- moved C1 1.80 mm to (22.9, 19.1)
- moved C2 1.80 mm to (16.5, 22.9)
- moved OK1 1.80 mm to (19.1, 11.4)
- moved R2 1.80 mm to (24.1, 25.4)
- moved R4 1.80 mm to (26.7, 6.35)
- moved C3 1.80 mm to (68.6, 8.89)
- moved DA2 1.80 mm to (33.0, 5.08)
- moved R5 1.80 mm to (44.5, 5.08)
- moved C4 1.80 mm to (55.9, 17.8)
- moved DA1 1.80 mm to (40.6, 17.8)
- moved R3 1.80 mm to (61.0, 15.2)
- moved X2 1.80 mm to (68.6, 19.1)
Other:
- board size 160 x 100 mm -> 74.9 x 30.1 mm
